File: Prj 1 - LED Tourch/Prj 1 - LED Tourch.kicad_pcb (KiCad board)
At the start: 2 copper layers, 71.4 x 23.6 mm, 4 parts, among them SW1 SW_DIP_x01

Commit message: add graphics and silkscreen
Parts:
- added REF**: KiCad-Logo2_8mm_SilkScreen, Symbol:KiCad-Logo2_8mm_SilkScreen, B.Cu at (153.2, 88.1)
Other:
- board text added: "+"
- board text added: "-"
- board text added: "V1.0"
