File: Prj 2 - Breadboard Power Supply/Prj 2 - Breadboard Power Supply.kicad_pcb (KiCad board)
At the start: 2 copper layers, 17 parts, among them J1 Conn_01x02_Pin, J2 Conn_01x03_Pin, J3 Conn_01x02_Pin, J4 Conn_01x03_Pin, J5 Screw_Terminal_01x02, J6 Barrel_Jack_Switch, J7 Screw_Terminal_01x02, U1 LM7805_TO220, U2 LM317_TO-220

Commit message: initial layout of the board
Parts:
- moved C2 98.0 mm to (116.1, 66.0)
- moved J4 92.9 mm to (120.1, 56.6), turned to 90 degrees
- moved C1 88.5 mm to (124.7, 66.0), turned to 180 degrees
- moved C3 84.9 mm to (121.9, 98.3)
- moved D1 81.5 mm to (134.3, 81.8)
- moved U2 79.9 mm to (118.4, 91.9)
- moved J2 78.4 mm to (118.9, 104.1), turned to 90 degrees
- moved U1 77.5 mm to (123.2, 70.9), turned to 180 degrees
- moved R2 72.1 mm to (137.8, 74.4), turned to 180 degrees
- moved R3 70.1 mm to (137.8, 92.5), turned to 180 degrees
- moved R1 70.1 mm to (137.8, 88.6), turned to 180 degrees
- moved S1 70.0 mm to (135.1, 68.3), turned to 180 degrees
- moved J6 68.4 mm to (129.4, 80.8)
- moved J1 67.1 mm to (142.2, 55.9)
- moved J5 64.7 mm to (130.8, 58.4)
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Other:
- board outline added: 35.6 x 52.6 mm
